Commit message: Изменение скрипта для практической работы

File: ROS_1/workspace/test_robot/urdf/simple_robot.urdf (robot description, URDF)
Before this commit: robot simple_robot, 3 links, 2 joints
Links:
- added link front_caster, mass 0.5; collision cylinder length=0.03 radius=0.05; visual cylinder length=0.03 radius=0.05
- link base_link: geometry collision box size=0.4 0.28 0.1; visual box size=0.4 0.28 0.1
- link left_wheel: geometry collision cylinder length=0.05 radius=0.1; visual cylinder length=0.05 radius=0.1
- link right_wheel: geometry collision cylinder length=0.05 radius=0.1; visual cylinder length=0.05 radius=0.1
Joints:
- added joint front_caster_joint: type continuous, parent base_link, child front_caster, origin xyz=0.18 0 0.05 rpy=0 0 0, axis 0 0 1
- joint left_wheel_joint: axis 0 1 0 -> 0 0 1; origin xyz=0 0.2 0 rpy=-1.5708 0 0 -> xyz=0 0.27 0 rpy=1.5708 0 0
- joint right_wheel_joint: axis 0 1 0 -> 0 0 1; origin xyz=0 -0.2 0 rpy=-1.5708 0 0 -> xyz=0 -0.27 0 rpy=1.5708 0 0
